File: AIS-Avionics-2026-2027/SRAD/Power Board - One per battery/Power Board - One per battery.kicad_sch (KiCad schematic)
At the start: 3 parts, among them J1 Conn_01x02, J2 Conn_01x02

Commit message: Updated SRAD power board for singular component
Parts:
- J1, J2: footprint Connector_JST:JST_PH_B2B-PH-K_1x02_P2.00mm_Vertical -> Reconfigured Standard Components:JST_PH_B2B-PH-K_1x02_P2.00mm_Vertical_CAD_Fixed
Changed lines of the file:
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@@
 			)
 		)
-		(property "Footprint" "Connector_JST:JST_PH_B2B-PH-K_1x02_P2.00mm_Vertical"
+		(property "Footprint" "Reconfigured Standard Components:JST_PH_B2B-PH-K_1x02_P2.00mm_Vertical_CAD_Fixed"
 			(at 182.88 99.06 0)
 			(effects
@@
 			)
 		)
-		(property "Footprint" "Connector_JST:JST_PH_B2B-PH-K_1x02_P2.00mm_Vertical"
+		(property "Footprint" "Reconfigured Standard Components:JST_PH_B2B-PH-K_1x02_P2.00mm_Vertical_CAD_Fixed"
 			(at 182.88 88.9 0)
 			(effects

Commit message: Battery shenanigans.
So many battery shenanigans
Parts:
- removed J1, J2: Conn_01x02, Reconfigured Standard Components:JST_PH_B2B-PH-K_1x02_P2.00mm_Vertical_CAD_Fixed, symbol Connector_Generic:Conn_01x02
- added D1: D, Package_TO_SOT_THT:TO-264-2_Vertical, symbol Device:D
- added F1: Fuse, Fuse:Fuseholder_Littelfuse_445_030_series_5x30mm, symbol Device:Fuse
- added J1, J2: Conn_01x02_Pin, Connector_JST:JST_PH_B2B-PH-K_1x02_P2.00mm_Vertical, symbol Connector:Conn_01x02_Pin
Connections:
- net at BT1.2 (-): now also J2.1 (Pin_1)
- net at BT1.1 (+): now also F1.2
- new net: D1.2 (A), F1.1
- new net: D1.1 (K), J1.2 (Pin_2)
- new net: J1.1 (Pin_1), J2.2 (Pin_2)
